File: hardware/RC-Multiswitch-Sound-ESP32-S3.kicad_pcb (KiCad board)
At the start: 2 copper layers, 106 x 68.2 mm, 38 parts, among them CN1 UART A, CN2 3S, CN4 Lautsprecher, J1 Ausgaenge, J11 TPA3118 HW-327, J2 PCM5102A, J5 UART B, J6 UART C, J9 microSD-TF-Modul, U1 ESP32-S3-DevKitC-1 (N16R8), U2 ULN2803A

Commit message: PCB: Martins Stand 20.10. (nach Prüfung C3/S3)
Parts:
- added G***: LOGO, LOGO, F.Cu at (226.7, 93.9)
